Commit message: changed many things rsp,rplidar,launch_sim,  added config files

File: mybot_description/urdf/mybot.xacro (robot description, xacro)
@@ -26,4 +26,12 @@
     </geometry>
   </collision>
+</link>
+<!-- Base Footprint Link -->
+<joint name="base_footprint_joint" type="fixed">
+  <parent link="baselink"/>
+  <child link="base_footprint"/>
+  <origin xyz="0 0 0" rpy="0 0 0"/>
+</joint>
+<link name="base_footprint">
 </link>
 <link name="lidar">

Commit message: display.launch

File: mybot_description/urdf/mybot.xacro (robot description, xacro)
@@ -26,12 +26,4 @@
     </geometry>
   </collision>
-</link>
-<!-- Base Footprint Link -->
-<joint name="base_footprint_joint" type="fixed">
-  <parent link="baselink"/>
-  <child link="base_footprint"/>
-  <origin xyz="0 0 0" rpy="0 0 0"/>
-</joint>
-<link name="base_footprint">
 </link>
 <link name="lidar">

Commit message: base_footprint

File: mybot_description/urdf/mybot.xacro (robot description, xacro)
@@ -27,4 +27,11 @@
   </collision>
 </link>
+  <joint name="base_footprint_joint" type="fixed">
+        <parent link="base_link"/>
+        <child link="base_footprint"/>
+        <origin xyz="0 0 0" rpy="0 0 0"/>
+    </joint>
+    <link name="base_footprint">
+    </link>
 <link name="lidar">
   <inertial>
